Commit message: Update FullAssemFIN.urdf

File: backend/Testing/FullAssemFIN.urdf (robot description, URDF)
Before this commit: robot FullAssemFIN, 31 links, 30 joints
Links:
- link Camera: geometry collision mesh filename=package://FullAssemFIN15/meshes/Camera.STL; visual mesh filename=package://FullAssemFIN15/meshes/Camera.STL
- link chest: mass 0.295734188674782 -> 0.419117350386115; geometry collision mesh filename=package://FullAssemFIN15/meshes/chest.STL; visual mesh filename=package://FullAssemFIN15/meshes/chest.STL
- link chest_back: geometry collision mesh filename=package://FullAssemFIN15/meshes/chest_back.STL; visual mesh filename=package://FullAssemFIN15/meshes/chest_back.STL
- link chest_front: mass 0.0836698829483839 -> 0.0836698829483879; geometry collision mesh filename=package://FullAssemFIN15/meshes/chest_front.STL; visual mesh filename=package://FullAssemFIN15/meshes/chest_front.STL
- link foot_left: mass 0.109810659435826 -> 0.109810659186526; geometry collision mesh filename=package://FullAssemFIN15/meshes/foot_left.STL; visual mesh filename=package://FullAssemFIN15/meshes/foot_left.STL
- link foot_right: mass 0.109792597961213 -> 0.109792588884947; geometry collision mesh filename=package://FullAssemFIN15/meshes/foot_right.STL; visual mesh filename=package://FullAssemFIN15/meshes/foot_right.STL
- link head: geometry collision mesh filename=package://FullAssemFIN15/meshes/head.STL; visual mesh filename=package://FullAssemFIN15/meshes/head.STL
- link hip_left_high: mass 0.0665008727926668 -> 0.066500872640875; geometry collision mesh filename=package://FullAssemFIN15/meshes/hip_left_high.STL; visual mesh filename=package://FullAssemFIN15/meshes/hip_left_high.STL
- link hip_left_in: mass 0.0712276180867603 -> 0.0712276180867601; geometry collision mesh filename=package://FullAssemFIN15/meshes/hip_left_in.STL; visual mesh filename=package://FullAssemFIN15/meshes/hip_left_in.STL
- link hip_left_low: mass 0.167133352428784 -> 0.16713334826647; geometry collision mesh filename=package://FullAssemFIN15/meshes/hip_left_low.STL; visual mesh filename=package://FullAssemFIN15/meshes/hip_left_low.STL
- link hip_right_high: mass 0.0665008726408751 -> 0.0665008726568549; geometry collision mesh filename=package://FullAssemFIN15/meshes/hip_right_high.STL; visual mesh filename=package://FullAssemFIN15/meshes/hip_right_high.STL
- link hip_right_in: geometry collision mesh filename=package://FullAssemFIN15/meshes/hip_right_in.STL; visual mesh filename=package://FullAssemFIN15/meshes/hip_right_in.STL
- link hip_right_low: mass 0.167468510508758 -> 0.167468511096326; geometry collision mesh filename=package://FullAssemFIN15/meshes/hip_right_low.STL; visual mesh filename=package://FullAssemFIN15/meshes/hip_right_low.STL
- link knee_left: mass 0.15114673120389 -> 0.151146730843275; geometry collision mesh filename=package://FullAssemFIN15/meshes/knee_left.STL; visual mesh filename=package://FullAssemFIN15/meshes/knee_left.STL
- link knee_right: mass 0.151146731235653 -> 0.151146730924696; geometry collision mesh filename=package://FullAssemFIN15/meshes/knee_right.STL; visual mesh filename=package://FullAssemFIN15/meshes/knee_right.STL
- link left_arm: mass 0.082113849315734 -> 0.205497013543678; geometry collision mesh filename=package://FullAssemFIN15/meshes/left_arm.STL; visual mesh filename=package://FullAssemFIN15/meshes/left_arm.STL
- link left_elbow: mass 0.145005574369976 -> 0.0817358599952458; geometry collision mesh filename=package://FullAssemFIN15/meshes/left_elbow.STL; visual mesh filename=package://FullAssemFIN15/meshes/left_elbow.STL
- link left_hand: mass 0.101380759300584 -> 0.041267310421405; geometry collision mesh filename=package://FullAssemFIN15/meshes/left_hand.STL; visual mesh filename=package://FullAssemFIN15/meshes/left_hand.STL
- link left_shoulder1: mass 0.133882143828078 -> 0.0104989821167456; geometry collision mesh filename=package://FullAssemFIN15/meshes/left_shoulder1.STL; visual mesh filename=package://FullAssemFIN15/meshes/left_shoulder1.STL
- link left_shoulder2: mass 0.140671760279634 -> 0.140671761076457; geometry collision mesh filename=package://FullAssemFIN15/meshes/left_shoulder2.STL; visual mesh filename=package://FullAssemFIN15/meshes/left_shoulder2.STL
- link left_wrist: mass 0.0853918664394992 -> 0.0252784174888945; geometry collision mesh filename=package://FullAssemFIN15/meshes/left_wrist.STL; visual mesh filename=package://FullAssemFIN15/meshes/left_wrist.STL
- link neck: geometry collision mesh filename=package://FullAssemFIN15/meshes/neck.STL; visual mesh filename=package://FullAssemFIN15/meshes/neck.STL
- link right_arm: mass 0.0821137195067692 -> 0.0821137195067691; geometry collision mesh filename=package://FullAssemFIN15/meshes/right_arm.STL; visual mesh filename=package://FullAssemFIN15/meshes/right_arm.STL
- link right_elbow: geometry collision mesh filename=package://FullAssemFIN15/meshes/right_elbow.STL; visual mesh filename=package://FullAssemFIN15/meshes/right_elbow.STL
- link right_hand: geometry collision mesh filename=package://FullAssemFIN15/meshes/right_hand.STL; visual mesh filename=package://FullAssemFIN15/meshes/right_hand.STL
- link right_shoulder1: geometry collision mesh filename=package://FullAssemFIN15/meshes/right_shoulder1.STL; visual mesh filename=package://FullAssemFIN15/meshes/right_shoulder1.STL
- link right_shoulder2: geometry collision mesh filename=package://FullAssemFIN15/meshes/right_shoulder2.STL; visual mesh filename=package://FullAssemFIN15/meshes/right_shoulder2.STL
- link right_wrist: geometry collision mesh filename=package://FullAssemFIN15/meshes/right_wrist.STL; visual mesh filename=package://FullAssemFIN15/meshes/right_wrist.STL
- link stomach: mass 0.112924078010695 -> 0.112924078010694; geometry collision mesh filename=package://FullAssemFIN15/meshes/stomach.STL; visual mesh filename=package://FullAssemFIN15/meshes/stomach.STL
- link stomach_low: mass 0.127534330377033 -> 0.127534330375141; geometry collision mesh filename=package://FullAssemFIN15/meshes/stomach_low.STL; visual mesh filename=package://FullAssemFIN15/meshes/stomach_low.STL
- link stomack_low_back: mass 0.147883656235969 -> 0.147883656236176; geometry collision mesh filename=package://FullAssemFIN15/meshes/stomack_low_back.STL; visual mesh filename=package://FullAssemFIN15/meshes/stomack_low_back.STL
Joints:
- joint Camera: origin xyz=0 0.10563 0.019299 rpy=1.5708 0.27854 3.1416 -> xyz=0.00129702055956225 0.101533990866758 -0.0770080285181508 rpy=-1.60490199320971 0 0
- joint chest_back: axis 0 1 0 -> 0 0 0; origin xyz=-0.01683 -0.0049556 0.21791 rpy=0.034104 0.010452 0.0065942 -> xyz=-0.015626 0.0041101 0.21852 rpy=0.034104 0.010452 0.0065942
- joint chest_front: axis 0 1 0 -> 0 0 0
- joint foot_left: axis -1 0 0 -> 1 0 0; limit lower=0 upper=0 effort=0 velocity=0 -> (none)
- joint foot_right: limit lower=0 upper=0 effort=0 velocity=0 -> (none); origin xyz=0 -0.21875 -0.01255 rpy=1.5708 0 3.1416 -> xyz=0 -0.21875 0.011588 rpy=1.5708 0 3.1416
- joint head: axis -0.020202 0.99922 0.034033 -> -1 0 0; limit lower=0 upper=0 effort=0 velocity=0 -> (none); origin xyz=0.0013216 0.052073 -0.1056 rpy=0 -0.00023277 0 -> xyz=0.020803 0 0 rpy=0 0 0
- joint hip_left_high: axis 0 1 0 -> 0 0 0; limit lower=0 upper=0 effort=0 velocity=0 -> (none)
- joint hip_left_in: axis 0 1 0 -> 0 0 0; limit lower=0 upper=0 effort=0 velocity=0 -> (none)
- joint hip_left_low: axis 0 -1 0 -> 0 0 0; limit lower=0 upper=0 effort=0 velocity=0 -> (none)
- joint hip_right_high: axis 0 1 0 -> 0 0 0; limit lower=0 upper=0 effort=0 velocity=0 -> (none)
- joint hip_right_in: axis 0 1 0 -> 0 0 0; limit lower=0 upper=0 effort=0 velocity=0 -> (none)
- joint hip_right_low: axis 0 0 0 -> 0 0 1; limit lower=0 upper=0 effort=0 velocity=0 -> (none); origin xyz=0.024482 0.2366 -0.0083418 rpy=0 -1.5318 -3.1416 -> xyz=0.00036231 0.0546 -0.0092832 rpy=0 -1.5318 -3.1416
- joint knee_left: axis 0 1 0 -> 0 0 0; limit lower=0 upper=0 effort=0 velocity=0 -> (none)
- joint knee_right: axis 0 0 -1 -> 0 0 1; limit lower=0 upper=0 effort=0 velocity=0 -> (none); origin xyz=0 -0.0019 0 rpy=0 0 0.015442 -> xyz=0 -0.1839 0 rpy=0 0 0.015442
- joint left_arm_twist: axis 0 1 0 -> -1 0 0; origin xyz=-0.026413 -0.0815 0.0128 rpy=0 0 0 -> xyz=0.00026682 -0.00075346 -0.048366 rpy=-1.5592 1.5555 -1.4879
- joint left_elbow: axis 0 1 0 -> -1 0 0; origin xyz=-0.0142 -0.044896 0.00012922 rpy=3.1416 0 -1.5708 -> xyz=0.10838 0.012907 0.00085871 rpy=1.5555 1.5368 1.5708
- joint left_hand: axis 0 1 0 -> -1 0 0; origin xyz=-0.018501 0.14157 0.0021722 rpy=-1.5714 0.0041657 2.9929 -> xyz=-0.078489 -0.0002665 0.014514 rpy=1.0976 -0.029908 -1.5708
- joint left_shoulder_raise: axis 1 0 0 -> -1 0.00071125 -0.0012765; origin xyz=-0.0066345 0.0367 0 rpy=0.025116 0 -3.1416 -> xyz=0.023528 0.00079477 -0.010776 rpy=1.543 -1.4993 -1.5528
- joint left_shoulder_twist: axis 0 -1 0 -> -1 0 0; origin xyz=0.062771 -0.012926 0.27864 rpy=0.0097647 0.034102 -1.5646 -> xyz=0.077364 -0.034143 0.27834 rpy=1.5707 -0.009759 0.0059046
- joint left_wrist: axis 0 1 0 -> -1 0 0; origin xyz=0.12738 -0.0138 0.002 rpy=0 0 -1.5708 -> xyz=1.9415E-05 0.0088059 0.13025 rpy=1.6049 1.5555 1.5708
- joint neck_turn: axis 0 1 0 -> -0.0015815 0.99926 -0.038308; limit lower=0 upper=0 effort=0 velocity=0 -> (none); origin xyz=-0.017795 -0.013377 0.29536 rpy=1.5367 0.009759 -3.1357 -> xyz=0.0037758 -0.018817 0.34931 rpy=1.5708 0.0097511 -3.1359
- joint right_arm_twist: limit lower=0 upper=0 effort=0 velocity=0 -> (none); origin xyz=-0.0815 0.019779 -0.0128 rpy=-3.1416 0 1.5708 -> xyz=-0.046932 0.019779 0 rpy=-3.1416 0 1.5708
- joint right_elbow: limit lower=0 upper=0 effort=0 velocity=0 -> (none); origin xyz=0.0142 -0.044896 0.00012922 rpy=0 0 -1.5708 -> xyz=0.0142 -0.079464 0.012929 rpy=0 0 -1.5708
- joint right_hand: limit lower=0 upper=0 effort=0 velocity=0 -> (none)
- joint right_shoulder_raise: axis 0 -1 0 -> 0 1 0; limit lower=0 upper=0 effort=0 velocity=0 -> (none)
- joint right_shoulder_twist: axis 0 1 0 -> 0 0 0; limit lower=0 upper=0 effort=0 velocity=0 -> (none); origin xyz=-0.098019 -0.013875 0.27707 rpy=-3.1318 0.034102 -1.5646 -> xyz=-0.096814 -0.0048096 0.27768 rpy=-3.1318 0.034102 -1.5646
- joint right_wrist: limit lower=0 upper=0 effort=0 velocity=0 -> (none)
- joint stomach: axis 0 1 0 -> 0 0 0; limit lower=0 upper=0 effort=0 velocity=0 -> (none)
- joint stomach_low: axis 1 0 0 -> 0 0 0; limit lower=0 upper=0 effort=0 velocity=0 -> (none)
- joint stomack_low_back: axis 0 -1 0 -> 0 0 0; limit lower=0 upper=0 effort=0 velocity=0 -> (none)
