Commit message: urdf limits commentted

File: backend/Testing/FullAssemFIN_tempProbe.urdf (robot description, URDF)
Before this commit: robot FullAssemFIN_tempProbe, 31 links, 30 joints
Joints:
- joint back: limit lower=0 upper=0 effort=0 velocity=0 -> (none)
- joint back_pelvic: limit lower=0 upper=0 effort=0 velocity=0 -> (none)
- joint camera: limit lower=0 upper=0 effort=0 velocity=0 -> (none)
- joint elbow_left: limit lower=0 upper=0 effort=0 velocity=0 -> (none)
- joint elbow_right: limit lower=0 upper=0 effort=0 velocity=0 -> (none)
- joint foot_left: limit lower=0 upper=0 effort=0 velocity=0 -> (none)
- joint foot_right: limit lower=0 upper=0 effort=0 velocity=0 -> (none)
- joint forearm_left: limit lower=0 upper=0 effort=0 velocity=0 -> (none)
- joint forearm_right: limit lower=0 upper=0 effort=0 velocity=0 -> (none)
- joint front_pelvic: limit lower=0 upper=0 effort=0 velocity=0 -> (none)
- joint hand_left: limit lower=0 upper=0 effort=0 velocity=0 -> (none)
- joint hand_right: limit lower=0 upper=0 effort=0 velocity=0 -> (none)
- joint head: limit lower=0 upper=0 effort=0 velocity=0 -> (none)
- joint hip_in_left: limit lower=0 upper=0 effort=0 velocity=0 -> (none)
- joint hip_in_right: limit lower=0 upper=0 effort=0 velocity=0 -> (none)
- joint hip_left: limit lower=0 upper=0 effort=0 velocity=0 -> (none)
- joint hip_out_left: limit lower=0 upper=0 effort=0 velocity=0 -> (none)
- joint hip_out_right: limit lower=0 upper=0 effort=0 velocity=0 -> (none)
- joint hip_right: limit lower=0 upper=0 effort=0 velocity=0 -> (none)
- joint knee_left: limit lower=0 upper=0 effort=0 velocity=0 -> (none)
- joint middle: limit lower=0 upper=0 effort=0 velocity=0 -> (none)
- joint neck: limit lower=0 upper=0 effort=0 velocity=0 -> (none)
- joint shoulder1_left: limit lower=0 upper=0 effort=0 velocity=0 -> (none)
- joint shoulder1_right: limit lower=0 upper=0 effort=0 velocity=0 -> (none)
- joint shoulder2_left: limit lower=0 upper=0 effort=0 velocity=0 -> (none)
- joint shoulder2_right: limit lower=0 upper=0 effort=0 velocity=0 -> (none)
- joint stomach: limit lower=0 upper=0 effort=0 velocity=0 -> (none)
- joint wrist_left: limit lower=0 upper=0 effort=0 velocity=0 -> (none)
- joint wrist_right: limit lower=0 upper=0 effort=0 velocity=0 -> (none)
