Commit message: update URDF limit and offset

File: backend/Testing/FullAssemFIN_straight_2025_5.urdf (robot description, URDF)
Before this commit: robot FullAssemFIN_straight_2025_5, 32 links, 31 joints
Joints:
- joint shoulder2_left: limit (none) -> lower=-1.628 upper=1.628 effort=0 velocity=0

Commit message: Update FullAssemFIN_straight_2025_5.urdf

File: backend/Testing/FullAssemFIN_straight_2025_5.urdf (robot description, URDF)
Before this commit: robot FullAssemFIN_straight_2025_5, 32 links, 31 joints
Joints:
- joint shoulder2_left: limit lower=-1.628 upper=1.628 effort=0 velocity=0 -> (none)
